File: 02-analog.kicad_sch (KiCad schematic)
At the start: 24 parts, among them J2 Superseal_1.0_5pol_MicA, J3 Superseal_1.0_5pol_MicB

Commit message: modified:   01-power.kicad_sch 	modified:   02-analog.kicad_sch 	modified:   03-adc.kicad_sch 	modified:   04-mcu.kicad_sch 	modified:   05-io.kicad_sch 	modified:   README.md 	modified:   exhaust-mic.kicad_pcb 	modified:   exhaust-mic.kicad_pro 	new file:   fp-lib-table 	modified:   lib/exhaust-mic.kicad_sym 	new file:   lib/exhaust-mic.pretty/Infineon_PG-LLGA-5-1.kicad_mod 	new file:   lib/exhaust-mic.pretty/TSSOP-30_4.4x7.8mm_P0.5mm.kicad_mod 	new file:   mic-head/fp-lib-table 	new file:   mic-head/mic-head.kicad_pcb 	modified:   mic-head/mic-head.kicad_pro 	modified:   mic-head/mic-head.kicad_sch 	modified:   output/bom-mainboard.csv 	modified:   output/bom-mic-head.csv 	new file:   output/main.net 	new file:   output/michead.net 	new file:   output/mikrofonkopf-gerber.zip 	new file:   output/mikrofonkopf-oben.svg 	new file:   output/mikrofonkopf-pcb.pdf 	new file:   output/mikrofonkopf-pos.csv 	new file:   output/mikrofonkopf-unten.svg 	modified:   tools/build_lib.py 	modified:   tools/build_main.py 	modified:   tools/build_mic_head.py 	new file:   tools/build_michead_pcb.py 	new file:   tools/build_outputs.py 	new file:   tools/build_pcb.py 	new file:   tools/pcbgen.py 	new file:   tools/pcbmap.py 	new file:   tools/route.py 	new file:   tools/verify.py
Parts:
- J2: value Superseal_1.0_5pol_MicA -> XH-5pol_MicA; footprint Connector_TE:TE_Superseal_1.0_5way -> Connector_JST:JST_XH_S5B-XH-A_1x05_P2.50mm_Horizontal; MPN (none) -> S5B-XH-A(LF)(SN)
- J3: value Superseal_1.0_5pol_MicB -> XH-5pol_MicB; footprint Connector_TE:TE_Superseal_1.0_5way -> Connector_JST:JST_XH_S5B-XH-A_1x05_P2.50mm_Horizontal; MPN (none) -> S5B-XH-A(LF)(SN)
- L2, L3: footprint Inductor_SMD:L_CommonModeChoke_Wuerth_WE-SL2 -> Inductor_SMD:L_CommonMode_Wuerth_WE-SL2
Changed lines of the file:
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@@
       (effects (font (size 1.27 1.27)))
     )
-    (property "Value" "Superseal_1.0_5pol_MicA" (at 45 83.89 0)
-      (effects (font (size 1.27 1.27)))
-    )
-    (property "Footprint" "Connector_TE:TE_Superseal_1.0_5way" (at 45 75 0)
+    (property "Value" "XH-5pol_MicA" (at 45 83.89 0)
+      (effects (font (size 1.27 1.27)))
+    )
+    (property "Footprint" "Connector_JST:JST_XH_S5B-XH-A_1x05_P2.50mm_Horizontal" (at 45 75 0)
       (effects (font (size 0.508 0.508)) hide)
     )
     (property "Datasheet" "" (at 45 75 0)
+      (effects (font (size 1.27 1.27)) hide)
+    )
+    (property "MPN" "S5B-XH-A(LF)(SN)" (at 45 75 0)
       (effects (font (size 1.27 1.27)) hide)
     )
@@
       (effects (font (size 1.27 1.27)))
     )
-    (property "Footprint" "Inductor_SMD:L_CommonModeChoke_Wuerth_WE-SL2" (at 140 82.62 0)
+    (property "Footprint" "Inductor_SMD:L_CommonMode_Wuerth_WE-SL2" (at 140 82.62 0)
       (effects (font (size 0.508 0.508)) hide)
     )
@@
       (effects (font (size 1.27 1.27)))
     )
-    (property "Value" "Superseal_1.0_5pol_MicB" (at 45 208.89 0)
-      (effects (font (size 1.27 1.27)))
-    )
-    (property "Footprint" "Connector_TE:TE_Superseal_1.0_5way" (at 45 200 0)
+    (property "Value" "XH-5pol_MicB" (at 45 208.89 0)
+      (effects (font (size 1.27 1.27)))
+    )
+    (property "Footprint" "Connector_JST:JST_XH_S5B-XH-A_1x05_P2.50mm_Horizontal" (at 45 200 0)
       (effects (font (size 0.508 0.508)) hide)
     )
     (property "Datasheet" "" (at 45 200 0)
+      (effects (font (size 1.27 1.27)) hide)
+    )
+    (property "MPN" "S5B-XH-A(LF)(SN)" (at 45 200 0)
       (effects (font (size 1.27 1.27)) hide)
     )
@@
       (effects (font (size 1.27 1.27)))
     )
-    (property "Footprint" "Inductor_SMD:L_CommonModeChoke_Wuerth_WE-SL2" (at 140 207.62 0)
-      (effects (font (size 0.508 0.508)) hide)
-    )
+    (property "Footprint" "Inductor_SMD:L_CommonMode_Wuerth_WE-SL2" (at 140 207.62 0)
+      (effects (font (size 0.508 0.508)) hide)
+    )
