File: 05-io.kicad_sch (KiCad schematic)
At the start: 34 parts, among them J6 GPS_unbestueckt, J7 I2C_Erweiterung, Q3 2N7002, Q4 2N7002, SW3 REC, SW4 MARK, U7 DS3231SN, U8 SN65HVD230D

Commit message: modified:   01-power.kicad_sch 	modified:   02-analog.kicad_sch 	modified:   03-adc.kicad_sch 	modified:   04-mcu.kicad_sch 	modified:   05-io.kicad_sch 	modified:   README.md 	modified:   exhaust-mic.kicad_pcb 	modified:   exhaust-mic.kicad_pro 	new file:   fp-lib-table 	modified:   lib/exhaust-mic.kicad_sym 	new file:   lib/exhaust-mic.pretty/Infineon_PG-LLGA-5-1.kicad_mod 	new file:   lib/exhaust-mic.pretty/TSSOP-30_4.4x7.8mm_P0.5mm.kicad_mod 	new file:   mic-head/fp-lib-table 	new file:   mic-head/mic-head.kicad_pcb 	modified:   mic-head/mic-head.kicad_pro 	modified:   mic-head/mic-head.kicad_sch 	modified:   output/bom-mainboard.csv 	modified:   output/bom-mic-head.csv 	new file:   output/main.net 	new file:   output/michead.net 	new file:   output/mikrofonkopf-gerber.zip 	new file:   output/mikrofonkopf-oben.svg 	new file:   output/mikrofonkopf-pcb.pdf 	new file:   output/mikrofonkopf-pos.csv 	new file:   output/mikrofonkopf-unten.svg 	modified:   tools/build_lib.py 	modified:   tools/build_main.py 	modified:   tools/build_mic_head.py 	new file:   tools/build_michead_pcb.py 	new file:   tools/build_outputs.py 	new file:   tools/build_pcb.py 	new file:   tools/pcbgen.py 	new file:   tools/pcbmap.py 	new file:   tools/route.py 	new file:   tools/verify.py
Parts:
- BT1: value CR2032 -> CR1220; footprint Battery:BatteryHolder_Keystone_3034_1x20mm -> Battery:BatteryHolder_Keystone_3000_1x12mm; MPN (none) -> Keystone 3000
Changed lines of the file:
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@@
       (effects (font (size 1.27 1.27)) (justify left))
     )
-    (property "Value" "CR2032" (at 143.1 77.745 0)
+    (property "Value" "CR1220" (at 143.1 77.745 0)
       (effects (font (size 1.27 1.27)) (justify left))
     )
-    (property "Footprint" "Battery:BatteryHolder_Keystone_3034_1x20mm" (at 140.56 75.84 0)
+    (property "Footprint" "Battery:BatteryHolder_Keystone_3000_1x12mm" (at 140.56 75.84 0)
       (effects (font (size 0.508 0.508)) hide)
     )
@@
       (effects (font (size 1.27 1.27)) hide)
     )
+    (property "MPN" "Keystone 3000" (at 140.56 75.84 0)
+      (effects (font (size 1.27 1.27)) hide)
+    )
