File: 05-io.kicad_sch (KiCad schematic)
At the start: 34 parts, among them J6 GPS_unbestueckt, J7 I2C_Erweiterung, Q3 2N7002, Q4 2N7002, SW3 REC, SW4 MARK, U7 DS3231SN, U8 SN65HVD230D

Commit message: modified:   01-power.kicad_sch 	modified:   02-analog.kicad_sch 	modified:   03-adc.kicad_sch 	modified:   04-mcu.kicad_sch 	modified:   05-io.kicad_sch 	modified:   exhaust-mic.kicad_pcb 	modified:   exhaust-mic.kicad_pro 	modified:   exhaust-mic.kicad_sch 	modified:   mic-head/mic-head.kicad_pcb 	modified:   mic-head/mic-head.kicad_pro 	modified:   mic-head/mic-head.kicad_sch 	new file:   ~exhaust-mic.kicad_pro.lck
Parts:
- BT1: value CR1220 -> CR2032; footprint Battery:BatteryHolder_Keystone_3000_1x12mm -> Battery:BatteryHolder_Keystone_3034_1x20mm; MPN Keystone 3000 -> (none)
- LS1: value Piezo_SMD -> Piezo; footprint Buzzer_Beeper:Buzzer_Murata_PKMCS0909E -> Buzzer_Beeper:Buzzer_12x9.5RM7.6; MPN PKMCS0909E4000-R1 -> (none)
Other:
- note removed: "DS3231SN mit integriertem TCXO: +/-2 ppm ueber -40...+85 C. Das ist die"
- note removed: "Der 1-Hz-Ausgang SQW rastet in der Firmware den Samplezaehler ein und"
- note removed: "Der ESP32-S3 hat TWAI, also klassisches CAN 2.0B bis 1 Mbit/s und"
- note removed: "Die Kamera nimmt Blitz oder Piep mit auf, danach laesst sich der Clip im"
- note removed: "EXT_BTN vom Harness liegt parallel zu SW4."
- note removed: "Interne Pull-ups des ESP32 genuegen; entprellt wird in Software."
- note removed: "J6: 1=3V3 2=TX 3=RX 4=PPS 5=GND"
- note removed: "J7: 1=3V3 2=SDA 3=SCL 4=GND"
- note removed: "LED_SYNC und der Piezo markieren den Aufnahmestart sichtbar und hoerbar."
- note removed: "R48 setzt die Flankensteilheit; 0R = maximale Bitrate."
- note removed: "Schnittprogramm framegenau ausrichten - das schafft keine Uhr allein."
- note removed: "Voraussetzung fuer brauchbare Zeitstempel im Motorradheck."
- note removed: "kein CAN-FD. Passend dazu ein 3,3-V-Transceiver - ein TCAN1051"
- note removed: "liefert damit eine driftfreie Zuordnung Uhrzeit zu Audiosample."
- note removed: "waere hier falsch, der braucht 5 V."
- company: Hayabusa / exhaust-mic -> (none)
- title: Exhaust-Mic - Echtzeituhr, CAN, Bedienung und Videosynchronisation -> Echtzeituhr, CAN, Bedienung und Videosynchronisation
- moved on the sheet: BT1, C50, C51, D22, J6, J7, LS1, Q3, Q4, R40, R41, R42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

Commit message: Beschaffungsdaten aus DigiKey in die vorhandenen Schaltplaene eintragen
Die Felder MPN, Hersteller und DigiKey werden nicht mehr geraten, sondern
gegen die Produktdatenbank ermittelt und mit Lagerfilter geprueft. Grundlage
sind die Schaltplandateien, wie sie auf der Platte liegen - die Generatoren
sind inzwischen aelter und wurden nicht angefasst.

tools/pick_digikey.py prueft jeden Treffer gegen die Parameter, die DigiKey
mitliefert: Kapazitaet, Spannungsfestigkeit, Dielektrikum, Widerstandswert,
Toleranz, Belastbarkeit, Bauform. Die Stichwortsuche allein reicht nicht -
auf "10 kOhm 1% 0603" antwortet DigiKey auch mit 11,5 k in 0201. Was aus der
Schaltung kommt und nicht in der Stueckliste steht, liegt in SPEC; Mechanik
und Steckverbinder in MANUELL; nicht lagernde Typen mit Ersatz und
Begruendung in ERSATZ.

tools/apply_digikey.py schreibt die Felder in die vorhandenen Dateien, ohne
sie neu zu erzeugen: vorhandene Werte werden ersetzt, neue Felder als
Abschrift des Datenblattfelds eingefuegt, damit Einrueckung und Schreibweise
passen. Vorhandene Hinweise bleiben stehen und werden ergaenzt. Mehrteilige
Bauteile bekommen die Felder an jedem Teil.

Ergebnis: 67 von 75 Positionen mit lagernder Herstellernummer, drei
brauchen kein Bauteil. Neun Positionen weichen auf einen gleichwertigen
Ersatz aus, weil der eingetragene Typ leer ist - Begruendung steht im Feld
Hinweis am Bauteil. Offen bleiben J1/J2/J3 (Superseal 1.0 gibt es bei
DigiKey nur kabelseitig), J4 (XKB-Steckverbinder nicht gefuehrt) und MK1
(IM73A135V01 ohne Bestand, kein Ersatz mit gleichem Gehaeuse).

ERC ist unveraendert; die Stuecklisten sind neu exportiert.
Parts:
- BT1: DigiKey (none) -> 36-3034CT-ND; Hersteller (none) -> Keystone Electronics; MPN (none) -> 3034TR
- C50, C51, C52: DigiKey (none) -> 1292-1642-1-ND; Hersteller (none) -> Walsin Technology Corporation; MPN (none) -> 0603B104K250CT
- D20: DigiKey (none) -> 160-LTST-C190GKTCT-ND; Hersteller (none) -> Lite-On Inc.; MPN (none) -> LTST-C190GKT
- D21: DigiKey (none) -> 160-1436-1-ND; Hersteller (none) -> Lite-On Inc.; MPN (none) -> LTST-C190KRKT
- D22: DigiKey (none) -> 160-2220-1-ND; Hersteller (none) -> Lite-On Inc.; MPN (none) -> LTW-170ZDC
- J6: DigiKey (none) -> 35-PREC005SAAN-RC-ND; Hersteller (none) -> Sullins Connector Solutions; MPN (none) -> PREC005SAAN-RC
- J7: DigiKey (none) -> 35-PREC004SAAN-RC-ND; Hersteller (none) -> Sullins Connector Solutions; MPN (none) -> PREC004SAAN-RC
- LS1: DigiKey (none) -> 668-AT-1240-TT-ND; Hersteller (none) -> PUI Audio, Inc.; MPN (none) -> AT-1240-TT
- Q3, Q4: DigiKey (none) -> T2N7002BKLMCT-ND; Hersteller (none) -> Toshiba Semiconductor and Storage; MPN (none) -> T2N7002BK,LM
- R40, R41: DigiKey (none) -> 311-4.70KHRCT-ND; Hersteller (none) -> YAGEO; MPN (none) -> RC0603FR-074K7L
- R42, R43, R44, R45, R46, R47, R48: DigiKey (none) -> 311-10.0KHRCT-ND; Hersteller (none) -> YAGEO; MPN (none) -> RC0603FR-0710KL
- R49: DigiKey (none) -> 738-RMCF0805FT120RCT-ND; Hersteller (none) -> Stackpole Electronics Inc; MPN (none) -> RMCF0805FT120R
- R50, R51, R52: DigiKey (none) -> 541-1.00KHCT-ND; Hersteller (none) -> Vishay Dale; MPN (none) -> CRCW06031K00FKEA
- R53: DigiKey (none) -> 2019-RK73H2ATTD18R0FCT-ND; Hersteller (none) -> KOA Speer Electronics, Inc.; MPN (none) -> RK73H2ATTD18R0F
- R54, R55: DigiKey (none) -> 311-100KHRCT-ND; Hersteller (none) -> YAGEO; MPN (none) -> RC0603FR-07100KL
- SW3, SW4: DigiKey (none) -> EG5470CT-ND; Hersteller (none) -> E-Switch; MPN (none) -> TL3342F260QG
- U7: DigiKey (none) -> DS3231SN#-ND; Hersteller (none) -> Analog Devices Inc./Maxim Integrated
- U8: DigiKey (none) -> 296-23353-5-ND; Hersteller (none) -> Texas Instruments; Hinweis (none) -> Ersatz fuer SN65HVD230DR: gleicher Baustein in Automotive-Q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; MPN SN65HVD230DR -> SN65HVD230QDG4Q1
