File: 04-mcu.kicad_sch (KiCad schematic)
At the start: 16 parts, among them J4 USB-C, J5 microSD_PushPush, SW1 RESET, SW2 BOOT, U6 ESP32-S3-WROOM-1-N8R2

Commit message: Footprints im Schaltplan auf den Stand des Layouts ziehen
Neun Bauteile trugen im Schaltplan einen Footprint, der so nicht baubar ist.
Das Layout hatte sie laengst ersetzt; jetzt steht es auch im Schaltplan:

  U5      TSSOP-30 4,4 x 9,7 / 0,65  ->  4,4 x 7,8 / 0,5  (Datenblatt)
  U6      ESP32-S2-WROOM             ->  ESP32-S3-WROOM-1
  L2, L3  L_CommonModeChoke_WE-SL2   ->  L_CommonMode_WE-SL2
  J1..J3  TE Superseal 1.0           ->  JST XH liegend
  BT1     Keystone 3034 / CR2032     ->  Keystone 3000 / CR1220
  LS1     Piezo bedrahtet 12 mm      ->  Murata-Landmuster 9 x 9 mm SMD

Wo sich damit das Bauteil aendert, sind Wert und Bestellnummer mitgezogen.
Zwei Punkte dabei zum Nachlesen:

* BT1 hat mit CR1220 rund ein Viertel der Kapazitaet von CR2032. Die
  Platine ist fuer den 12-mm-Halter gebohrt, darum folgt der Schaltplan.
* Der im Layout benannte Murata PKMCS0909E ist abgekuendigt ("Last Time
  Buy") und nur fuer 1,5 V spezifiziert, angesteuert wird aber mit 3,3 V.
  Bestellt wird darum ein 3-V-Typ gleicher Bauform (Same Sky
  CPT-9019A-SMT-TR); das Landmuster gehoert gegen das Datenblatt geprueft.

Damit sind die Steckverbinder J1..J3 beschaffbar - Superseal 1.0 gibt es bei
DigiKey nur kabelseitig. Offen bleiben noch J4 und MK1.

Schaltplanparitaet: 18 -> 9 Abweichungen auf der Hauptplatine, 2 auf dem
Mikrofonkopf. Die restlichen sind keine Footprints mehr, sondern Symbole:
U2 hat einen Pin 4, den das SOT-223 nicht hat, und dem microSD-Symbol fehlt
der Schirmanschluss. Beides steht im README.

Die Stueckliste fuehrt jetzt eine Spalte Hinweis - dort landen die
Ersatzgruende, die vorher nur im Schaltplan standen.

DRC unveraendert: 0 Fehler, 10 Warnungen, 7 offene Verbindungen. ERC
unveraendert. Stuecklisten, Fertigungsdaten und PDFs neu erzeugt.
Parts:
- U6: footprint RF_Module:ESP32-S2-WROOM -> RF_Module:ESP32-S3-WROOM-1
Changed lines of the file:
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@@
 			)
 		)
-		(property "Footprint" "RF_Module:ESP32-S2-WROOM"
+		(property "Footprint" "RF_Module:ESP32-S3-WROOM-1"
 			(at 165.1 144.78 0)
 			(hide yes)
