File: 04-mcu.kicad_sch (KiCad schematic)
At the start: 16 parts, among them J4 USB-C, J5 microSD_PushPush, SW1 RESET, SW2 BOOT, U6 ESP32-S3-WROOM-1-N8R2

Commit message: Die beiden Symbolfehler geradeziehen, die der Abgleich meldete
U2: Das Symbol exhaust-mic:TLV1117LV33 hatte vier Pins. Das SOT-223 hat drei
Anschluesse und eine Kuehlfahne, die innen an Pin 2 haengt - Pin 4 gab es
nie. Er lag am selben Netz wie Pin 2, elektrisch also folgenlos. Entfernt
sind der Pin aus der Symbolkopie und aus dem Bauteil sowie die beiden
Draehte und der Verbindungspunkt, die ihn an Pin 2 gefuehrt haben. Damit
faellt auch der ERC-Fehler "Stromausgang gegen Stromausgang" weg.

J5: Micro_SD_Card_Det1 kennt einen Schaltkontakt und legt den Schirm auf
Pin 10. Der Kartenhalter DM3D-SF hat zwei Schaltkontakte auf Pad 9 und 10
und den Schirm auf Pad 11 - das passt zu Micro_SD_Card_Det2. Die
gemeinsamen Pins liegen dort an denselben Stellen, die vorhandene
Verdrahtung bleibt also unangetastet; der neue Pin 10 (DET_A) ist ueber
zwei Draehte an den vorhandenen Massepunkt gelegt.

Schaltplanparitaet 9 -> 4 Abweichungen, und die vier sind die
Befestigungsbohrungen H1..H4, die absichtlich kein Symbol haben. Auf dem
Mikrofonkopf dasselbe Bild mit H1 und H2.

ERC 4 -> 3 Fehler. Die restlichen drei sind power_pin_not_driven an +4V6,
AVDD und VBAT: an diesen Netzen fehlt ein PWR_FLAG.

DRC unveraendert: 0 Fehler, 10 Warnungen, 7 offene Verbindungen.
Stueckliste, Fertigungsdaten und PDF neu erzeugt.
Parts:
- J5: symbol Connector:Micro_SD_Card_Det1 -> Connector:Micro_SD_Card_Det2
Connections:
- net GND: now also J5.11 (SHIELD)
Changed lines of the file:
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@@
 		)
+	)
+	(wire
+		(pts
+			(xy 317.24 209.94) (xy 308.35 209.94)
+		)
+		(stroke
+			(width 0)
+			(type default)
+		)
+	)
+	(wire
+		(pts
+			(xy 308.35 209.94) (xy 308.35 212.48)
+		)
+		(stroke
+			(width 0)
+			(type default)
+		)
+	)
+	(junction
+		(at 308.35 212.48)
+		(diameter 0)
+		(color 0 0 0 0)
 	)
 	(symbol
@@
 	)
 	(symbol
-		(lib_id "Connector:Micro_SD_Card_Det1")
+		(lib_id "Connector:Micro_SD_Card_Det2")
 		(at 340.1 199.78 0)
 		(unit 1)
@@
 		(pin "10"
 		)
+		(pin "11"
+		)
 		(instances

Commit message: J4 auf den GCT USB4085-GF-A umstellen und das Layout nachziehen
Den XKB-Typ zum bisherigen Footprint fuehrt DigiKey nicht. Der GCT
USB4085-GF-A ist lagernd (80 000 Stueck), kostet 0,78 EUR - aber es ist
keine gleiche Bauform: der XKB klebt mit einer Padreihe oben auf, der GCT
steckt mit sechzehn Anschluessen in zwei versetzten Reihen durch die
Platine. Am Motorrad ist das mechanisch die bessere Wahl; dafuer sperren
die Bohrungen alle vier Lagen.

tools/swap_footprint.py (neu) tauscht den Footprint auf der Platine und
ordnet die Netze ueber die Padnamen aus der Netzliste zu. Danach ist der
Autorouter einmal komplett durchgelaufen: 5 offene Verbindungen statt der
7 vorher, und keine davon auf einem Signalnetz - es sind nur noch
Masseflaechen-Stuecke auf der Rueckseite.

tools/trim_warnings.py (neu) raeumt lose Bahnenden und zu dicht gesetzte
Bohrungen weg, die KiCad nur als Warnung meldet. Einzeln, mit Rueckprobe:
pauschales Loeschen hat die Zahl der offenen Verbindungen von 5 auf 6
gehoben, weil ein als "lose" gemeldetes Stueck nach dem Fuellen der
Flaechen doch getragen hat. fix_drc.py kann jetzt ebenfalls Warnungen
mitnehmen (--alle), taugt dafuer aber nur mit Vorsicht.

Zwei echte Fehler in handroute.py behoben, die dabei auffielen:

* Bahnenden auf einer Innenlage wurden als "auf allen Lagen erreichbar"
  gelesen, weil das Muster nur F.Cu und B.Cu kannte. Ergebnis war eine
  Leiterbahn auf der Aussenlage zu einem Ende, das dort gar nicht liegt -
  Kupfer, das nichts verbindet, und ein Werkzeug, das Erfolg meldet.
* Der Anschlussdraht einer neu gesetzten Durchkontaktierung landete immer
  auf F.Cu oder B.Cu, egal wo das Bahnende lag.

Ausserdem darf handroute jetzt auf allen Signallagen ziehen, nicht nur auf
den beiden aeusseren; die durchgehende Masseflaeche auf In1 bleibt tabu.
route.py loest das Arbeitsverzeichnis absolut auf - mit relativer Angabe
fand Java das Jar nicht, weil freerouting mit dem Arbeitsverzeichnis als
cwd laeuft.

Zwei Bauteile sind im Lauf d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
Parts:
- J4: footprint Connector_USB:USB_C_Receptacle_XKB_U262-16XN-4BVC11 -> Connector_USB:USB_C_Receptacle_GCT_USB4085; DigiKey (none) -> 2073-USB4085-GF-ACT-ND; Hersteller (none) -> GCT; Hinweis (none) -> durchkontaktiert statt SMD; den XKB-Typ zum vorherigen Foot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; MPN (none) -> USB4085-GF-A
Changed lines of the file:
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@@
 			)
 		)
-		(property "Footprint" "Connector_USB:USB_C_Receptacle_XKB_U262-16XN-4BVC11"
+		(property "Footprint" "Connector_USB:USB_C_Receptacle_GCT_USB4085"
 			(at 330.2 80.01 0)
 			(hide yes)
@@
 			(show_name no)
 			(do_not_autoplace no)
+			(effects
+				(font
+					(size 1.27 1.27)
+				)
+			)
+		)
+		(property "MPN" "USB4085-GF-A"
+			(at 330.2 80.01 0)
+			(hide yes)
+			(show_name no)
+			(do_not_autoplace no)
+			(effects
+				(font
+					(size 1.27 1.27)
+				)
+			)
+		)
+		(property "Hersteller" "GCT"
+			(at 330.2 80.01 0)
+			(hide yes)
+			(show_name no)
+			(do_not_autoplace no)
+			(effects
+				(font
+					(size 1.27 1.27)
+				)
+			)
+		)
+		(property "DigiKey" "2073-USB4085-GF-ACT-ND"
+			(at 330.2 80.01 0)
+			(hide yes)
+			(show_name no)
+			(do_not_autoplace no)
+			(effects
+				(font
+					(size 1.27 1.27)
+				)
+			)
+		)
+		(property "Hinweis" "durchkontaktiert statt SMD; den XKB-Typ zum vorherigen Footprint fuehrt DigiKey nicht"
+			(at 330.2 80.01 0)
+			(hide yes)
+			(show_name no)
+			(do_not_autoplace no)

Commit message: modified:   01-power.kicad_sch 	modified:   04-mcu.kicad_sch 	modified:   README.md 	modified:   docs/beschaffung.md 	modified:   docs/entwicklung.md 	modified:   exhaust-mic.kicad_pcb 	modified:   firmware/README.md 	modified:   firmware/main/CMakeLists.txt 	modified:   firmware/main/main.c 	modified:   firmware/main/pins.h 	new file:   firmware/main/zuendung.c 	new file:   firmware/main/zuendung.h 	modified:   firmware/tools/pins_aus_netzliste.py 	modified:   output/bilder/hauptplatine-bottom.png 	modified:   output/bilder/hauptplatine-top.png 	modified:   output/bom-mainboard.csv 	modified:   output/exhaust-mic-schaltplan.pdf 	modified:   output/hauptplatine-gerber.zip 	modified:   output/hauptplatine-oben.svg 	modified:   output/hauptplatine-pcb.pdf 	modified:   output/hauptplatine-pos.csv 	modified:   output/hauptplatine-unten.svg 	modified:   output/main.net
Connections:
- net PWR_HOLD: now reaches U6.35 (IO42)
- no-connect marks 6 -> 5
Changed lines of the file:
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@@
 	)
 	(no_connect
-		(at 180.34 157.48)
-	)
-	(no_connect
 		(at 180.34 160.02)
 	)
@@
 				)
 			)
+		)
+	)
+	(wire
+		(pts
+			(xy 180.34 157.48) (xy 199.39 157.48)
+		)
+		(stroke
+			(width 0)
+			(type default)
+		)
+	)
+	(global_label "PWR_HOLD"
+		(shape output)
+		(at 199.39 157.48 0)
+		(fields_autoplaced yes)
+		(effects
+			(font
+				(size 1.27 1.27)
+			)
+			(justify left)
+		)
+		(property "Intersheetrefs" "${INTERSHEET_REFS}"
+			(at 199.39 157.48 0)
+			(hide yes)
+			(show_name no)
+			(do_not_autoplace no)
+			(effects
+				(font
+					(size 1.27 1.27)
+				)
+			)
