File: exhaust-mic.kicad_pcb (KiCad board)
At the start: 4 copper layers, 72 x 55 mm, 131 parts, among them J1 JST_XH_6pol, J2 JST_XH_5pol_MicA, J3 JST_XH_5pol_MicB, J4 USB-C, J5 microSD_PushPush, J6 GPS_unbestueckt, J7 I2C_Erweiterung, Q1 SI2309CDS, Q3 2N7002, Q4 2N7002, SW1 RESET, SW2 BOOT, SW3 REC, SW4 MARK, U1 LM5164DDA, U2 NCP1117ST33, U3 LP5907MFX-3.3, U5 PCM1863DBT, U6 ESP32-S3-WROOM-1-N8R2, U7 DS3231SN, U8 SN65HVD230Q, Y1 24.576MHz

Commit message: J4 auf den GCT USB4085-GF-A umstellen und das Layout nachziehen
Den XKB-Typ zum bisherigen Footprint fuehrt DigiKey nicht. Der GCT
USB4085-GF-A ist lagernd (80 000 Stueck), kostet 0,78 EUR - aber es ist
keine gleiche Bauform: der XKB klebt mit einer Padreihe oben auf, der GCT
steckt mit sechzehn Anschluessen in zwei versetzten Reihen durch die
Platine. Am Motorrad ist das mechanisch die bessere Wahl; dafuer sperren
die Bohrungen alle vier Lagen.

tools/swap_footprint.py (neu) tauscht den Footprint auf der Platine und
ordnet die Netze ueber die Padnamen aus der Netzliste zu. Danach ist der
Autorouter einmal komplett durchgelaufen: 5 offene Verbindungen statt der
7 vorher, und keine davon auf einem Signalnetz - es sind nur noch
Masseflaechen-Stuecke auf der Rueckseite.

tools/trim_warnings.py (neu) raeumt lose Bahnenden und zu dicht gesetzte
Bohrungen weg, die KiCad nur als Warnung meldet. Einzeln, mit Rueckprobe:
pauschales Loeschen hat die Zahl der offenen Verbindungen von 5 auf 6
gehoben, weil ein als "lose" gemeldetes Stueck nach dem Fuellen der
Flaechen doch getragen hat. fix_drc.py kann jetzt ebenfalls Warnungen
mitnehmen (--alle), taugt dafuer aber nur mit Vorsicht.

Zwei echte Fehler in handroute.py behoben, die dabei auffielen:

* Bahnenden auf einer Innenlage wurden als "auf allen Lagen erreichbar"
  gelesen, weil das Muster nur F.Cu und B.Cu kannte. Ergebnis war eine
  Leiterbahn auf der Aussenlage zu einem Ende, das dort gar nicht liegt -
  Kupfer, das nichts verbindet, und ein Werkzeug, das Erfolg meldet.
* Der Anschlussdraht einer neu gesetzten Durchkontaktierung landete immer
  auf F.Cu oder B.Cu, egal wo das Bahnende lag.

Ausserdem darf handroute jetzt auf allen Signallagen ziehen, nicht nur auf
den beiden aeusseren; die durchgehende Masseflaeche auf In1 bleibt tabu.
route.py loest das Arbeitsverzeichnis absolut auf - mit relativer Angabe
fand Java das Jar nicht, weil freerouting mit dem Arbeitsverzeichnis als
cwd laeuft.

Zwei Bauteile sind im Lauf d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
Parts:
- J4: footprint Connector_USB:USB_C_Receptacle_XKB_U262-16XN-4BVC11 -> Connector_USB:USB_C_Receptacle_GCT_USB4085
- moved J4 4.77 mm to (172.9, 71.6)
Routing:
- net GND: track 18.2 -> 71.9 mm, vias 822 -> 821
- net USB_DP: track 61.4 -> 90.3 mm
- net +3V3D: track 213.2 -> 220.5 mm
- net Net-(J4-CC2): track 60.2 -> 57.9 mm
- net USB_DM: track 72.4 -> 70.9 mm, vias 2 -> 1
- net +4V6: track 80.8 -> 82.3 mm
- net VBAT12: track 78.3 -> 79.5 mm
- net Net-(D20-K): track 4.76 -> 5.80 mm
- net Net-(D21-K): track 4.76 -> 5.52 mm
- net LED_SYNC: track 64.1 -> 64.8 mm
- net CANL: track 19.5 -> 20.1 mm
- net I2S_LRCK: track 59.2 -> 59.7 mm
- net Net-(D1-A): track 9.22 -> 9.75 mm
- net BUZZ: track 74.2 -> 74.7 mm
- net Net-(U5-VREF): track 2.71 -> 3.24 mm
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